File: Schematic-PCB/FT2232H_USB_to_JTAG_and_UART/FT2232H_USB_to_JTAG_and_UART.kicad_pcb (KiCad board)
At the start: 2 copper layers, 16 parts, among them J1 TI_JTAG14 Connector, J2 Conn_01x04_Pin, U1 FT2232H, U2 ISO7761, U3 ISO7221, U4 SN74ALVC244

Commit message: Removed buffer IC from schematic
Parts:
- removed U4: SN74ALVC244, SOIC-DIP:SOIC_20-DIP
- added J3: Conn_01x05_Pin, Connector_PinHeader_2.54mm:PinHeader_1x05_P2.54mm_Vertical, F.Cu at (154.3, 50.3)
- moved U2 21.6 mm to (121.4, 109.3)
- moved J1 16.1 mm to (147.5, 111.7)
- moved J2 6.48 mm to (164.4, 103.7), turned to 90 degrees
Connections:
- net GND1 renamed FTDI_GND
- U1 pad 31: unconnected-(U1-CS-Pad31) -> EEPROM_CS
- U1 pad 32: unconnected-(U1-CLK-Pad32) -> EEPROM_CLK
- U1 pad 33: unconnected-(U1-Data-Pad33) -> EEPROM_Data
- U2 pad 10: MID_TDO -> MCU_TDO
- U2 pad 12: MID_TMS -> MCU_TMS
- U2 pad 13: MID_TCK -> MCU_TCK
- U2 pad 14: MID_TRSTn -> MCU_TRSTn
- U2 pad 15: MID_TDI -> MCU_TDI
Routing:
- net MCU_TDO: track 103.3 -> 39.6 mm, vias 2 -> 0
- net EEPROM_Data: track 0.00 -> 50.2 mm, vias 0 -> 4
- net EEPROM_CLK: track 0.00 -> 49.6 mm, vias 0 -> 4
- net MCU_GND: track 173.7 -> 131.1 mm
- net EEPROM_CS: track 0.00 -> 40.6 mm, vias 0 -> 4
- net MCU_TCK: track 64.3 -> 30.5 mm, vias 2 -> 0
- net MID_TDI: track 32.9 -> 0.00 mm
- net MCU_VCC: track 85.6 -> 53.3 mm, vias 4 -> 2
- net +3.3V: track 218.5 -> 245.7 mm
- net MCU_TMS: track 79.5 -> 53.0 mm, vias 0 -> 2
- net MID_TRSTn: track 25.9 -> 0.00 mm
- net FT_TCK: track 67.9 -> 46.1 mm
- net FT_TDO: track 57.3 -> 36.5 mm
- net MID_TCK: track 20.3 -> 0.00 mm
- net MCU_TRSTn: track 57.2 -> 38.6 mm
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